Commit message: Fixed mesh offset in gripper .xarco

File: robot_ws/src/pkgs_from_moodle/wsg50_gripper/urdf/wsg_50.urdf.xacro (robot description, xacro)
@@ -73,5 +73,5 @@
   <link name="${name}_finger_left">
       <visual>
-	      <origin xyz="0.0 0 0" rpy="0 0 0" />
+	      <origin xyz="0.0 0 -0.22" rpy="0 0 0" />
          <geometry>
             <!--mesh filename="package://wsg_50_simulation/meshes/WSG-FMF.stl" scale="0.001 0.001 0.001"/-->
@@ -84,5 +84,5 @@
       <collision>
           <!--origin xyz="0 0 0.1" rpy="0 0 0" /-->
-	      <origin xyz="0 0 0" rpy="0 0 0" />
+	      <origin xyz="0 0 -0.22" rpy="0 0 0" />
          <geometry>
             <!--<mesh filename="package://wsg_50_simulation/meshes/WSG-FMF.stl" scale="0.001 0.001 0.001"/>-->
@@ -137,5 +137,5 @@
       <visual>
          <!--origin xyz="0.0 0 0.1" rpy="0 0 0" /-->
-	      <origin xyz="0.0 0 0" rpy="0 0 0" />
+	      <origin xyz="0.0 0 -0.22" rpy="0 0 0" />
          <geometry>
             <!--mesh filename="package://wsg_50_simulation/meshes/WSG-FMF.stl" scale="0.001 0.001 0.001"/-->
@@ -148,5 +148,5 @@
       <collision>
          <!--origin xyz="0 0 0.1" rpy="0 0 0" /-->
-         <origin xyz="0 0 0" rpy="0 0 0" />
+         <origin xyz="0 0 -0.22" rpy="0 0 0" />
          <geometry>
             <!--mesh filename="package://wsg_50_simulation/meshes/WSG-FMF.stl" scale="0.001 0.001 0.001"/-->

Commit message: Assignment 1 done

File: robot_ws/src/pkgs_from_moodle/wsg50_gripper/urdf/wsg_50.urdf.xacro (robot description, xacro)
@@ -73,5 +73,5 @@
   <link name="${name}_finger_left">
       <visual>
-	      <origin xyz="0.0 0 0" rpy="0 0 0" />
+	      <origin xyz="0.0 0 -${finger_length}" rpy="0 0 0" />
          <geometry>
             <!--mesh filename="package://wsg_50_simulation/meshes/WSG-FMF.stl" scale="0.001 0.001 0.001"/-->
@@ -84,5 +84,5 @@
       <collision>
           <!--origin xyz="0 0 0.1" rpy="0 0 0" /-->
-	      <origin xyz="0 0 0" rpy="0 0 0" />
+	      <origin xyz="0 0 -${finger_length}" rpy="0 0 0" />
          <geometry>
             <!--<mesh filename="package://wsg_50_simulation/meshes/WSG-FMF.stl" scale="0.001 0.001 0.001"/>-->
@@ -137,5 +137,5 @@
       <visual>
          <!--origin xyz="0.0 0 0.1" rpy="0 0 0" /-->
-	      <origin xyz="0.0 0 0" rpy="0 0 0" />
+	      <origin xyz="0.0 0 -${finger_length}" rpy="0 0 0" />
          <geometry>
             <!--mesh filename="package://wsg_50_simulation/meshes/WSG-FMF.stl" scale="0.001 0.001 0.001"/-->
@@ -148,5 +148,5 @@
       <collision>
          <!--origin xyz="0 0 0.1" rpy="0 0 0" /-->
-         <origin xyz="0 0 0" rpy="0 0 0" />
+         <origin xyz="0 0 -${finger_length}" rpy="0 0 0" />
          <geometry>
             <!--mesh filename="package://wsg_50_simulation/meshes/WSG-FMF.stl" scale="0.001 0.001 0.001"/-->
