Commit message: Created a separate package for modified gripper and deleted the original one

File: robot_ws/src/my_pkgs/dual_arm_robot/urdf/sia20d_with_wsg.xacro (robot description, xacro)
@@ -3,5 +3,5 @@
 	<xacro:macro name="motoman_sia20d_with_wsg" params="prefix">
 		<xacro:include filename="$(find motoman_sia20d_support)/urdf/sia20d_macro.xacro"/>
-		<xacro:include filename="$(find wsg50_gripper)/urdf/wsg_50.urdf.xacro"/>
+		<xacro:include filename="$(find wsg50_gripper_modified)/urdf/wsg_50_modified.urdf.xacro"/>
 		<xacro:motoman_sia20d prefix="${prefix}sia20d_"/>
 		<xacro:wsg_50_xacro name="${prefix}wsg" finger_length="0.22" finger_tip="0.0"/>

File: robot_ws/src/my_pkgs/wsg50_gripper_modified/urdf/wsg_50_modified.urdf.xacro (robot description, xacro)
@@ -10,5 +10,5 @@
          <origin xyz="0.0 0 0" rpy="0 0 0" />
          <geometry>
-            <mesh filename="package://wsg50_gripper/meshes/WSG50_110.stl" scale="1 1 1"/>
+            <mesh filename="package://wsg50_gripper_modified/meshes/WSG50_110.stl" scale="1 1 1"/>
          </geometry>
          <material name="grey">
@@ -19,5 +19,5 @@
           <origin xyz="0.0 0 0" rpy="0 0 0" />
           <geometry>
-             <mesh filename="package://wsg50_gripper/meshes/WSG50_110.stl" scale="1 1 1"/>
+             <mesh filename="package://wsg50_gripper_modified/meshes/WSG50_110.stl" scale="1 1 1"/>
          </geometry>
      </collision>
@@ -48,5 +48,5 @@
           <origin xyz="0.0 0 0" rpy="0 0 0" />
           <geometry>
-             <mesh filename="package://wsg50_gripper/meshes/GUIDE_WSG50_110.stl" scale="0.001 0.001 0.001"/>
+             <mesh filename="package://wsg50_gripper_modified/meshes/GUIDE_WSG50_110.stl" scale="0.001 0.001 0.001"/>
 	     <!--box size="0.0175 0.03 0.024"/-->
           </geometry>
@@ -59,5 +59,5 @@
           <geometry>
 	     <!--box size="0.0175 0.03 0.024"/-->
-             <mesh filename="package://wsg50_gripper/meshes/GUIDE_WSG50_110.stl" scale="0.001 0.001 0.001"/>
+             <mesh filename="package://wsg50_gripper_modified/meshes/GUIDE_WSG50_110.stl" scale="0.001 0.001 0.001"/>
          </geometry>
      </collision>
@@ -76,5 +76,5 @@
          <geometry>
             <!--mesh filename="package://wsg_50_simulation/meshes/WSG-FMF.stl" scale="0.001 0.001 0.001"/-->
-            <mesh filename="package://wsg50_gripper/meshes/REMODEL_finger.stl" scale="1 1 1"/>
+            <mesh filename="package://wsg50_gripper_modified/meshes/REMODEL_finger.stl" scale="1 1 1"/>
          </geometry>
          <material name="black">
@@ -87,5 +87,5 @@
          <geometry>
             <!--<mesh filename="package://wsg_50_simulation/meshes/WSG-FMF.stl" scale="0.001 0.001 0.001"/>-->
-	         <mesh filename="package://wsg50_gripper/meshes/REMODEL_finger.stl" scale="1 1 1"/>
+	         <mesh filename="package://wsg50_gripper_modified/meshes/REMODEL_finger.stl" scale="1 1 1"/>
          </geometry>
      </collision>
@@ -111,5 +111,5 @@
          <origin xyz="0.0 0 0" rpy="0 0 0" />
          <geometry>
-            <mesh filename="package://wsg50_gripper/meshes/GUIDE_WSG50_110.stl" scale="0.001 0.001 0.001"/>
+            <mesh filename="package://wsg50_gripper_modified/meshes/GUIDE_WSG50_110.stl" scale="0.001 0.001 0.001"/>
 	         <!--box size="0.0175 0.03 0.024"/-->
          </geometry>
@@ -122,5 +122,5 @@
          <geometry>
             <!--box size="0.0175 0.03 0.024"/-->
-            <mesh filename="package://wsg50_gripper/meshes/GUIDE_WSG50_110.stl" scale="0.001 0.001 0.001"/>
+            <mesh filename="package://wsg50_gripper_modified/meshes/GUIDE_WSG50_110.stl" scale="0.001 0.001 0.001"/>
          </geometry>
       </collision>
@@ -140,5 +140,5 @@
          <geometry>
             <!--mesh filename="package://wsg_50_simulation/meshes/WSG-FMF.stl" scale="0.001 0.001 0.001"/-->
-            <mesh filename="package://wsg50_gripper/meshes/REMODEL_finger.stl" scale="1 1 1"/>
+            <mesh filename="package://wsg50_gripper_modified/meshes/REMODEL_finger.stl" scale="1 1 1"/>
          </geometry>
          <material name="black">
@@ -151,5 +151,5 @@
          <geometry>
             <!--mesh filename="package://wsg_50_simulation/meshes/WSG-FMF.stl" scale="0.001 0.001 0.001"/-->
-	         <mesh filename="package://wsg50_gripper/meshes/REMODEL_finger.stl" scale="1 1 1"/>
+	         <mesh filename="package://wsg50_gripper_modified/meshes/REMODEL_finger.stl" scale="1 1 1"/>
          </geometry>
      </collision>

Commit message: Changed finger_length value to zero and changed back to using original wsg package (as was done in model answer)

File: robot_ws/src/my_pkgs/dual_arm_robot/urdf/sia20d_with_wsg.xacro (robot description, xacro)
@@ -3,11 +3,14 @@
 	<xacro:macro name="motoman_sia20d_with_wsg" params="prefix">
 		<xacro:include filename="$(find motoman_sia20d_support)/urdf/sia20d_macro.xacro"/>
-		<xacro:include filename="$(find wsg50_gripper_modified)/urdf/wsg_50_modified.urdf.xacro"/>
+		<!--<xacro:include filename="$(find wsg50_gripper_modified)/urdf/wsg_50_modified.urdf.xacro"/>-->
+		<xacro:include filename="$(find wsg50_gripper)/urdf/wsg_50.urdf.xacro"/>
 		<xacro:motoman_sia20d prefix="${prefix}sia20d_"/>
-		<xacro:wsg_50_xacro name="${prefix}wsg" finger_length="0.22" finger_tip="0.0"/>
+		<!--<xacro:wsg_50_xacro name="${prefix}wsg" finger_length="0.22" finger_tip="0.0"/>-->
+		<xacro:wsg_50_xacro name="${prefix}wsg" finger_length="0.0" finger_tip="0.0"/>
 		<joint name="${prefix}tool0-wsg" type="fixed">
 			<parent link="${prefix}sia20d_tool0"/>
 			<child link="${prefix}wsg_base_link"/>
-			<origin xyz="0 0 0" rpy="0 0 -3.1415926535"/>
+			<!--<origin xyz="0 0 0" rpy="0 0 -3.1415926535"/>-->
+			<origin xyz="0 0 0" rpy="0 0 0"/>
 		</joint>
 	</xacro:macro>

File: robot_ws/src/original_wsg_packages/wsg50_gripper/urdf/wsg_50.urdf.xacro (robot description, xacro)
@@ -10,5 +10,5 @@
          <origin xyz="0.0 0 0" rpy="0 0 0" />
          <geometry>
-            <mesh filename="package://wsg50_gripper_modified/meshes/WSG50_110.stl" scale="1 1 1"/>
+            <mesh filename="package://wsg50_gripper/meshes/WSG50_110.stl" scale="1 1 1"/>
          </geometry>
          <material name="grey">
@@ -19,5 +19,5 @@
           <origin xyz="0.0 0 0" rpy="0 0 0" />
           <geometry>
-             <mesh filename="package://wsg50_gripper_modified/meshes/WSG50_110.stl" scale="1 1 1"/>
+             <mesh filename="package://wsg50_gripper/meshes/WSG50_110.stl" scale="1 1 1"/>
          </geometry>
      </collision>
@@ -48,5 +48,5 @@
           <origin xyz="0.0 0 0" rpy="0 0 0" />
           <geometry>
-             <mesh filename="package://wsg50_gripper_modified/meshes/GUIDE_WSG50_110.stl" scale="0.001 0.001 0.001"/>
+             <mesh filename="package://wsg50_gripper/meshes/GUIDE_WSG50_110.stl" scale="0.001 0.001 0.001"/>
 	     <!--box size="0.0175 0.03 0.024"/-->
           </geometry>
@@ -59,5 +59,5 @@
           <geometry>
 	     <!--box size="0.0175 0.03 0.024"/-->
-             <mesh filename="package://wsg50_gripper_modified/meshes/GUIDE_WSG50_110.stl" scale="0.001 0.001 0.001"/>
+             <mesh filename="package://wsg50_gripper/meshes/GUIDE_WSG50_110.stl" scale="0.001 0.001 0.001"/>
          </geometry>
      </collision>
@@ -73,9 +73,8 @@
   <link name="${name}_finger_left">
       <visual>
-      	 <!--<origin xyz="0.0 0 -${finger_length}" rpy="0 0 0" /-->
-	     <origin xyz="0.0 0 0" rpy="0 0 0" />
+	      <origin xyz="0.0 0 0" rpy="0 0 0" />
          <geometry>
             <!--mesh filename="package://wsg_50_simulation/meshes/WSG-FMF.stl" scale="0.001 0.001 0.001"/-->
-            <mesh filename="package://wsg50_gripper_modified/meshes/REMODEL_finger.stl" scale="1 1 1"/>
+            <mesh filename="package://wsg50_gripper/meshes/REMODEL_finger.stl" scale="1 1 1"/>
          </geometry>
          <material name="black">
@@ -85,9 +84,8 @@
       <collision>
           <!--origin xyz="0 0 0.1" rpy="0 0 0" /-->
-          <!--<origin xyz="0 0 -${finger_length}" rpy="0 0 0" /-->
 	      <origin xyz="0 0 0" rpy="0 0 0" />
          <geometry>
             <!--<mesh filename="package://wsg_50_simulation/meshes/WSG-FMF.stl" scale="0.001 0.001 0.001"/>-->
-	         <mesh filename="package://wsg50_gripper_modified/meshes/REMODEL_finger.stl" scale="1 1 1"/>
+	         <mesh filename="package://wsg50_gripper/meshes/REMODEL_finger.stl" scale="1 1 1"/>
          </geometry>
      </collision>
@@ -113,5 +111,5 @@
          <origin xyz="0.0 0 0" rpy="0 0 0" />
          <geometry>
-            <mesh filename="package://wsg50_gripper_modified/meshes/GUIDE_WSG50_110.stl" scale="0.001 0.001 0.001"/>
+            <mesh filename="package://wsg50_gripper/meshes/GUIDE_WSG50_110.stl" scale="0.001 0.001 0.001"/>
 	         <!--box size="0.0175 0.03 0.024"/-->
          </geometry>
@@ -124,5 +122,5 @@
          <geometry>
             <!--box size="0.0175 0.03 0.024"/-->
-            <mesh filename="package://wsg50_gripper_modified/meshes/GUIDE_WSG50_110.stl" scale="0.001 0.001 0.001"/>
+            <mesh filename="package://wsg50_gripper/meshes/GUIDE_WSG50_110.stl" scale="0.001 0.001 0.001"/>
          </geometry>
       </collision>
@@ -139,9 +137,8 @@
       <visual>
          <!--origin xyz="0.0 0 0.1" rpy="0 0 0" /-->
-         <!--<origin xyz="0.0 0 -${finger_length}" rpy="0 0 0" /-->
 	      <origin xyz="0.0 0 0" rpy="0 0 0" />
          <geometry>
             <!--mesh filename="package://wsg_50_simulation/meshes/WSG-FMF.stl" scale="0.001 0.001 0.001"/-->
-            <mesh filename="package://wsg50_gripper_modified/meshes/REMODEL_finger.stl" scale="1 1 1"/>
+            <mesh filename="package://wsg50_gripper/meshes/REMODEL_finger.stl" scale="1 1 1"/>
          </geometry>
          <material name="black">
@@ -151,9 +148,8 @@
       <collision>
          <!--origin xyz="0 0 0.1" rpy="0 0 0" /-->
-         <!--<origin xyz="0 0 -${finger_length}" rpy="0 0 0" /-->
          <origin xyz="0 0 0" rpy="0 0 0" />
          <geometry>
             <!--mesh filename="package://wsg_50_simulation/meshes/WSG-FMF.stl" scale="0.001 0.001 0.001"/-->
-	         <mesh filename="package://wsg50_gripper_modified/meshes/REMODEL_finger.stl" scale="1 1 1"/>
+	         <mesh filename="package://wsg50_gripper/meshes/REMODEL_finger.stl" scale="1 1 1"/>
          </geometry>
      </collision>
